Commit message: treads

File: urdf/rover.urdf (robot description, URDF)
Before this commit: robot rover, 5 links, 4 joints
Links:
- link front_left_wheel: geometry collision cylinder length=0.07 radius=0.08; visual box size=0.006 0.052 0.055
- link front_right_wheel: geometry collision cylinder length=0.07 radius=0.08; visual box size=0.006 0.052 0.055
- link rear_left_wheel: geometry collision cylinder length=0.07 radius=0.08; visual box size=0.006 0.052 0.055
- link rear_right_wheel: geometry collision cylinder length=0.07 radius=0.08; visual box size=0.006 0.052 0.055
